Commit message: cartpole example (WIP)

File: raisim_gym/env/env/cartpole/cartpole/cartpole.urdf (robot description, URDF)
Before this commit: robot cartpole, 4 links, 3 joints
Links:
- link pole: geometry collision box size=0.05 0.05 0.0; visual box size=0.05 0.05 0.0
Joints:
- joint cart_to_pole: limit (none) -> lower=-6.28 upper=6.28 effort=80 velocity=15

Commit message: WIP...

File: raisim_gym/env/env/cartpole/cartpole/cartpole.urdf (robot description, URDF)
Before this commit: robot cartpole, 4 links, 3 joints
Links:
- link pole: geometry collision box size=0.05 0.05 1.0; visual box size=0.05 0.05 1.0
Joints:
- joint world_to_slider: origin xyz=0.0 0.0 0.0 -> xyz=0.0 0.0 1.0

Commit message: for debugging when reward reports inf.

File: raisim_gym/env/env/cartpole/cartpole/cartpole.urdf (robot description, URDF)
Before this commit: robot physics, 4 links, 3 joints
Links:
- link cart: geometry visual box size=0.5 0.5 0.2
- link pole: geometry visual box size=0.05 0.05 1.0
Joints:
- joint world_to_slider: origin xyz=0.0 0.0 1.0 -> xyz=0.0 0.0 5.0
